File: MatrixBoard2.kicad_sch (KiCad schematic)
At the start: 196 parts, among them J1 Conn_01x03_Male, J2 Conn_01x03_Male

Commit message: fixing footprints
Parts:
- D1, D10, D11, D12, D13, D14, D15, D16, D17, D18, D19, D2, D20, D21, D22, D23, D24, D25, D26, D27, D28, D29, D3, D30, D31, D32, D33, D34, D35, D36, D37, D38, D39, D4, D40, D41, D42, D43, D44, D45, D46, D47, D48, D49, D5, D50, D51, D52, D53, D54, D55, D56, D57, D58, D59, D6, D60, D61, D62, D63, D64, D65, D66, D67, D68, D69, D7, D70, D71, D72, D73, D74, D75, D76, D77, D78, D79, D8, D80, D81, D82, D83, D84, D85, D86, D87, D88, D89, D9, D90, D91, D92, D93, D94, D95, D96: footprint LED_SMD:LED_SK6812MINI_PLCC4_3.5x3.5mm_P1.75mm -> tightstuff:LED_SK6812MINI_PLCC4_3.5x3.5mm_P1.75mm

Commit message: Added possible Bulk Capacitance...
Parts:
- added C100, C101, C102, C103, C104, C97, C98, C99: 100uf, Capacitor_Tantalum_SMD:CP_EIA-6032-28_Kemet-C_Pad2.25x2.35mm_HandSolder, symbol Device:C_Polarized
Connections:
- net +5V: now also C100.1, C101.1, C102.1, C103.1, C104.1, C97.1, C98.1, C99.1
- net GND: now also C100.2, C101.2, C102.2, C103.2, C104.2, C97.2, C98.2, C99.2
Other:
- note added: "Bulk Capacitance... Warning: reversing polarity makes booms. Also: May not be needed."
- note added: "Decoupling Capacitance These may not ALL be required..."

Commit message: A bunch of cosmetic changes... (Mostly silkscreen OCD)
Connections:
- net GND: now also J1.3 (Pin_3), J2.3 (Pin_3); no longer J1.1 (Pin_1), J2.1 (Pin_1)
- net at R1.2: now also J1.1 (Pin_1); no longer J1.3 (Pin_3)
- net at R2.2: now also J2.1 (Pin_1); no longer J2.3 (Pin_3)
Changed lines of the file:
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@@
     (pin "2")
   )
-  (symbol (lib_id "Connector:Conn_01x03_Male") (at 21.59 24.13 0) (unit 1)
+  (symbol (lib_id "Connector:Conn_01x03_Male") (at 21.59 24.13 0) (mirror x) (unit 1)
     (in_bom yes) (on_board yes) (fields_autoplaced)
-    (property "Reference" "J1" (id 0) (at 22.225 16.51 0))
-    (property "Value" "Conn_01x03_Male" (id 1) (at 22.225 19.05 0))
+    (property "Reference" "J1" (id 0) (at 20.32 24.1299 0)
+      (effects (font (size 1.27 1.27)) (justify right))
+    )
+    (property "Value" "Conn_01x03_Male" (id 1) (at 20.32 25.3999 0)
+      (effects (font (size 1.27 1.27)) (justify right) hide)
+    )
     (property "Footprint" "Connector_PinHeader_2.54mm:PinHeader_1x03_P2.54mm_Vertical" (id 2) (at 21.59 24.13 0)
       (effects (font (size 1.27 1.27)) hide)
@@
     (pin "4")
   )
-  (symbol (lib_id "Connector:Conn_01x03_Male") (at 135.89 181.61 0) (unit 1)
+  (symbol (lib_id "Connector:Conn_01x03_Male") (at 135.89 181.61 0) (mirror x) (unit 1)
     (in_bom yes) (on_board yes) (fields_autoplaced)
-    (property "Reference" "J2" (id 0) (at 136.525 173.99 0))
-    (property "Value" "Conn_01x03_Male" (id 1) (at 136.525 176.53 0))
+    (property "Reference" "J2" (id 0) (at 134.62 181.6099 0)
+      (effects (font (size 1.27 1.27)) (justify right))
+    )
+    (property "Value" "Conn_01x03_Male" (id 1) (at 134.62 182.8799 0)
+      (effects (font (size 1.27 1.27)) (justify right) hide)
+    )
     (property "Footprint" "Connector_PinHeader_2.54mm:PinHeader_1x03_P2.54mm_Vertical" (id 2) (at 135.89 181.61 0)
       (effects (font (size 1.27 1.27)) hide)

Commit message: Did a bit o research into SK6812mini versions...
Parts:
- R1, R2: value 500 -> 510
Changed lines of the file:
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@@
     (in_bom yes) (on_board yes)
     (property "Reference" "R1" (id 0) (at 34.29 24.13 90))
-    (property "Value" "500" (id 1) (at 34.29 29.21 90))
+    (property "Value" "510" (id 1) (at 34.29 29.21 90))
     (property "Footprint" "Resistor_SMD:R_0805_2012Metric" (id 2) (at 34.29 24.892 90)
       (effects (font (size 1.27 1.27)) hide)
@@
     (in_bom yes) (on_board yes)
     (property "Reference" "R2" (id 0) (at 148.59 181.61 90))
-    (property "Value" "500" (id 1) (at 148.59 186.69 90))
+    (property "Value" "510" (id 1) (at 148.59 186.69 90))
     (property "Footprint" "Resistor_SMD:R_0805_2012Metric" (id 2) (at 148.59 182.372 90)
       (effects (font (size 1.27 1.27)) hide)
@@
     )
     (path "/46517f4f-933a-456e-a041-0e9aa98522b9"
-      (reference "R1") (unit 1) (value "500") (footprint "Resistor_SMD:R_0805_2012Metric")
+      (reference "R1") (unit 1) (value "510") (footprint "Resistor_SMD:R_0805_2012Metric")
     )
     (path "/be3c26cf-aa20-456b-805e-b92b209e1cb2"
-      (reference "R2") (unit 1) (value "500") (footprint "Resistor_SMD:R_0805_2012Metric")
+      (reference "R2") (unit 1) (value "510") (footprint "Resistor_SMD:R_0805_2012Metric")
     )
   )
